File: Flash PCB/puente H/puente H.kicad_sch (KiCad schematic)
At the start: 6 parts, among them IC1 TB6612FNG, J1 HEADER_8, J3 HEADER_8

Commit message: Arreglando errores de diseño
Parts:
- C3: footprint Capacitor_Tantalum_SMD:CP_EIA-2012-12_Kemet-R_Pad1.30x1.05mm_HandSolder -> Capacitor_Tantalum_SMD:CP_EIA-3528-21_Kemet-B_Pad1.50x2.35mm_HandSolder
Changed lines of the file:
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@@
       (effects (font (size 1.27 1.27)) (justify left))
     )
-    (property "Footprint" "Capacitor_Tantalum_SMD:CP_EIA-2012-12_Kemet-R_Pad1.30x1.05mm_HandSolder" (at 120.65 50.8 0)
+    (property "Footprint" "Capacitor_Tantalum_SMD:CP_EIA-3528-21_Kemet-B_Pad1.50x2.35mm_HandSolder" (at 120.65 50.8 0)
       (effects (font (size 1.27 1.27)) hide)
     )

Commit message: Arreglando Puente H
Parts:
- J1, J3: footprint Connector_PinSocket_2.00mm:PinSocket_1x08_P2.00mm_Vertical -> EESTN5:Pin_Header_Angled_1x08
Changed lines of the file:
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@@
       (effects (font (size 1.524 1.524)) (justify left))
     )
-    (property "Footprint" "Connector_PinSocket_2.00mm:PinSocket_1x08_P2.00mm_Vertical" (at 190.5 66.04 0)
+    (property "Footprint" "EESTN5:Pin_Header_Angled_1x08" (at 190.5 66.04 0)
       (effects (font (size 1.524 1.524)) hide)
     )
@@
       (effects (font (size 1.524 1.524)))
     )
-    (property "Footprint" "Connector_PinSocket_2.00mm:PinSocket_1x08_P2.00mm_Vertical" (at 92.71 104.14 0)
-      (effects (font (size 1.524 1.524)) hide)
-    )
+    (property "Footprint" "EESTN5:Pin_Header_Angled_1x08" (at 92.71 104.14 0)
+      (effects (font (size 1.524 1.524)) hide)
+    )
