File: Flash PCB/Plaqueta Mani/Plaqueta Mani/Plaqueta Mani.kicad_sch (KiCad schematic)
At the start: 1 part, among them J1 Arduino_Nano_Header

Commit message: Arreglando errores de diseño
Parts:
- J1: footprint EESTN5:arduino_nano_header -> (none)
Changed lines of the file:
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@@
 (kicad_sch (version 20230121) (generator eeschema)
   (paper "A4")
-  (symbol (lib_id "EESTN5:Arduino_Nano_Header") (at 132.334 72.644 0) (unit 1)
+  (symbol (lib_id "EESTN5:Arduino_Nano_Header") (at 145.796 82.042 0) (unit 1)
     (in_bom yes) (on_board yes) (dnp no) (fields_autoplaced)
-    (property "Reference" "J1" (at 132.334 45.72 0)
+    (property "Reference" "J1" (at 145.796 58.42 0)
       (effects (font (size 1.524 1.524)))
     )
-    (property "Value" "Arduino_Nano_Header" (at 132.334 48.26 0)
+    (property "Value" "Arduino_Nano_Header" (at 145.796 60.96 0)
       (effects (font (size 1.524 1.524)))
     )
-    (property "Footprint" "EESTN5:arduino_nano_header" (at 132.334 50.8 0)
+    (property "Footprint" "" (at 145.796 82.042 0)
       (effects (font (size 1.524 1.524)))
     )
-    (property "Datasheet" "" (at 132.334 72.644 0)
+    (property "Datasheet" "" (at 145.796 82.042 0)
       (effects (font (size 1.524 1.524)))
     )
@@
     (pin "9")
     (instances
-      (project "Flash Forma"
-        (path "/17d5f0a9-f2e8-4c5a-bea9-93a856536820"
+      (project "Plaqueta Mani"
+        (path "/b1c9236c-08e5-42c5-bca3-c7d41737a702"
           (reference "J1") (unit 1)
         )

Commit message: PLaqueta Mani Milton
Parts:
- added J2: VIN_BATTERY, Connector_PinHeader_2.00mm:PinHeader_1x02_P2.00mm_Vertical, symbol Connector:Conn_01x02_Pin
- added J3: VOUT_R, Connector_PinHeader_2.00mm:PinHeader_1x02_P2.00mm_Vertical, symbol Connector:Conn_01x02_Pin
- added J4: MOTOR1, EESTN5:BORNERA2_AZUL, symbol Connector:Conn_01x02_Pin
- added Jr1: MOTOR2, EESTN5:BORNERA2_AZUL, symbol Connector:Conn_01x02_Pin
- added P1: CONN_01X08, EESTN5:Pin_Header_Straight_1x08, symbol EESTN5:CONN_01X08
- added P2, P3: CONN_01X08, EESTN5:Socket_Strip_Straight_1x08, symbol EESTN5:CONN_01X08
- J1: footprint (none) -> Module:Arduino_Nano
Connections:
- net BI1: now reaches J1.10 (D7/AIN1)
- net BI1: now also P3.4 (P4)
- net STBY: now reaches J1.11 (D8/ICP)
- net STBY: now also P3.5 (P5)
- net AI1: now reaches J1.12 (D9/0C1)
- net AI1: now also P3.6 (P6)
- net AI2: now reaches J1.13 (D10/SS)
- net AI2: now also P3.7 (P7)
- net PWMA: now reaches J1.14 (D11/MOSI)
- net PWMA: now also P3.8 (P8)
- net QR_1: now reaches J1.19 (A0)
- net QR_1: now also P1.3 (P3)
- net QR_2: now reaches J1.20 (A1)
- net QR_2: now also P1.4 (P4)
- net QR_3: now reaches J1.21 (A2)
- net QR_3: now also P1.5 (P5)
- net QR_4: now reaches J1.22 (A3)
- net QR_4: now also P1.6 (P6)
- net QR_5: now reaches J1.23 (A4)
- net QR_5: now also P1.7 (P7)
- net QR_6: now reaches J1.24 (A5)
- net QR_6: now also P1.8 (P8)
- net +5V: now reaches J1.27 (5V)
- net +5V: now also P1.1 (P1), P2.2 (P2)
- net Earth: now reaches J1.29 (GND)
- net Earth: now also J1.4 (GND), J2.2 (Pin_2), J3.2 (Pin_2), P1.2 (P2), P2.3 (P3), P2.8 (P8), P3.1 (P1)
- net +7.5V: now reaches J1.30 (VIN)
- net +7.5V: now also J2.1 (Pin_1), J3.1 (Pin_1), P2.1 (P1)
- net PWMB: now reaches J1.8 (D5/T1)
- net PWMB: now also P3.2 (P2)
- net BI2: now reaches J1.9 (D6/AIN0)
- net BI2: now also P3.3 (P3)
- new net AO1: J4.2 (Pin_2), P2.4 (P4)
- new net AO2: J4.1 (Pin_1), P2.5 (P5)
- new net BO1: Jr1.1 (Pin_1), P2.7 (P7)
- new net BO2: Jr1.2 (Pin_2), P2.6 (P6)
Other:
- moved on the sheet: J1
