File: Plaqueta mani/Plaqueta mani.kicad_pcb (KiCad board)
At the start: 2 copper layers, 99.9 x 92.7 mm, 33 parts, among them J1 Arduino_Nano_Header, J1 HEADER_8, J2 Alimentacion +5v, J3 HEADER_8, J5 Motor A, J6 Motor B, P1 Modulo Qre113, P1 Modulo_QRE113, SW2 SW_SPDT, U1 QRE1113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

Commit message: Add files via upload
Parts:
- removed H1 (x2), H2 (x2), H3, H4: Mounting_Hole, EESTN5:hole_3mm
- removed P1: Modulo_QRE113, EESTN5:Socket_Strip_Angled_1x08
- removed P1: Modulo Qre113, EESTN5:Pin_Header_Straight_1x08
- added C1: 0.1uf, EESTN5:CAP_0.2, F.Cu at (159.8, 31.3)
- added C2: 0.1uf, EESTN5:CAP_0.2, F.Cu at (94.5, 31.3)
- added C3: C, EESTN5:CAP_ELEC_10X8mm, F.Cu at (151.6, 38.2)
- J2: value Alimentacion +5v -> Alimentacion +7.5v
- moved J2 103.1 mm to (159.9, 46.9), turned to 38.3 degrees
- moved J5 102.2 mm to (166.7, 31.3)
- moved J6 102.2 mm to (87.6, 31.3)
- moved J1 93.6 mm to (126.7, 64.4)
- moved SW2 93.1 mm to (138.8, 40.3)
- moved J3 92.4 mm to (117.7, 32.8)
- moved J1 92.4 mm to (117.8, 48.8)
- moved R10 8.85 mm to (144.4, 194.9)
- moved R2 8.85 mm to (106.0, 194.9)
- moved R5 8.85 mm to (122.3, 194.9)
- moved R7 8.85 mm to (138.8, 194.9)
- moved R9 8.85 mm to (155.8, 194.9)
- moved U1 8.85 mm to (100.4, 194.8)
- moved U3 8.85 mm to (116.6, 194.9)
- moved R4 8.85 mm to (80.5, 194.7)
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Connections:
- J1 pad 20: /QR_6 -> /QR_1
- J1 pad 21: /QR_5 -> /QR_2
- J1 pad 22: /QR_4 -> /QR_3
- J1 pad 23: /QR_3 -> /QR_4
- J1 pad 24: /QR_2 -> /QR_5
- J1 pad 25: /QR_1 -> /QR_6
- J1 pad 27: unconnected-(J1-5V-Pad27) -> +5V
- J1 pad 30: +5V -> +7.5V
Routing:
- net /QR_5: track 34.1 -> 137.3 mm
- net /QR_6: track 48.2 -> 149.7 mm
- net +5V: track 269.1 -> 368.7 mm, vias 0 -> 7
- net /QR_4: track 27.3 -> 126.0 mm
- net /QR_3: track 40.0 -> 134.9 mm
- net /QR_2: track 52.3 -> 147.0 mm
- net /QR_1: track 62.7 -> 157.3 mm
- net +7.5V: track 22.0 -> 59.3 mm
- net /BO1: track 37.1 -> 27.7 mm
- net /BO2: track 38.4 -> 31.2 mm
- net /AO1: track 56.5 -> 51.8 mm
- net Net-(SW2-A): track 27.4 -> 31.6 mm
- net /BI2: track 10.7 -> 7.93 mm
- net /AO2: track 57.4 -> 55.1 mm
- net /STBY: track 10.2 -> 7.94 mm
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Other:
- board size 99.9 x 92.7 mm -> 119.5 x 188.6 mm

Commit message: Agregue leds y actualice los pads del plaqueta mani
Parts:
- removed the J1 at (117.8, 48.8)
- removed the J1 at (126.7, 64.4)
- added J1: Arduino_Nano_Header, EESTN5:arduino_nano_header, F.Cu at (140.2, 63.1)
- added J1: HEADER_8, EESTN5:Pin_Header_Angled_1x08, F.Cu at (131.3, 47.6)
- added LED1: LED, EESTN5:LED_1206, F.Cu at (115.8, 67.0)
- added LED2: LED, EESTN5:LED_1206, F.Cu at (115.8, 59.2)
- moved C3 13.6 mm to (165.2, 36.9)
- moved J6 13.6 mm to (101.2, 30.0)
- moved SW2 13.6 mm to (152.3, 39.0)
- moved U4 13.6 mm to (146.9, 193.6)
- moved U5 13.6 mm to (163.8, 193.6)
- moved R12 13.6 mm to (174.7, 193.7)
- moved R8 13.6 mm to (140.8, 193.7)
- moved U6 13.6 mm to (180.8, 193.7)
- moved C2 13.6 mm to (108.0, 30.0)
- moved J3 13.6 mm to (131.2, 31.5)
- moved R1 13.6 mm to (108.8, 193.5)
- moved R3 13.6 mm to (104.1, 193.5)
- moved R4 13.6 mm to (94.1, 193.4)
- moved U1 13.6 mm to (113.9, 193.6)
- moved U2 13.6 mm to (99.0, 193.3)
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Routing:
- net /LED_1: track 0.00 -> 40.0 mm, vias 0 -> 1
- net /LED_2: track 0.00 -> 21.2 mm, vias 0 -> 1
- net +5V: track 368.7 -> 366.5 mm
- net /QR_1: track 157.3 -> 158.1 mm
- net /QR_2: track 147.0 -> 147.8 mm
- net /QR_3: track 134.9 -> 135.6 mm
- net Earth: vias 0 -> 1
Other:
- board size 119.5 x 188.6 mm -> 119.4 x 188.6 mm
