File: Plaqueta mani/Plaqueta mani.kicad_sch (KiCad schematic)
At the start: 35 parts, among them J1 Arduino_Nano_Header, J2 Alimentacion +5v, J3 Conn_01x02, J4 Conn_01x02, J5 Motor A, J6 Motor B, P1 Modulo_QRE113, P2 CONN_01X08, P3 CONN_01X08, P4 Modulo Qre113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

Commit message: Add files via upload
Parts:
- removed H1, H2, H3, H4, H5, H6: Mounting_Hole, EESTN5:hole_3mm, symbol EESTN5:Mounting_Hole
- removed J3, J4: Conn_01x02, EESTN5:Pin_Header_2, symbol Connector_Generic:Conn_01x02
- removed P1: Modulo_QRE113, EESTN5:Socket_Strip_Angled_1x08, symbol EESTN5:CONN_01X08
- added C1, C2: 0.1uf, EESTN5:CAP_0.2, symbol EESTN5:C
- added C3: C, EESTN5:CAP_ELEC_10X8mm, symbol EESTN5:C
- J2: value Alimentacion +5v -> Alimentacion +7.5v
- R11, R12, R3, R4, R7, R8: value 1k -> 10k
Connections:
- net +5V: now also J1.27 (5V); no longer J1.30 (VIN)
- net +7.5V: now also J1.30 (VIN)
- net AO1: now also C1.2
- net AO2: now also C1.1
- net BO1: now also C2.2
- net BO2: now also C2.1
- net Earth: now also C3.1
- net QR_1: now also J1.20 (A1); no longer J1.25 (A6)
- net QR_2: now also J1.21 (A2); no longer J1.24 (A5)
- net QR_3: now also J1.22 (A3); no longer J1.23 (A4)
- net QR_4: now also J1.23 (A4); no longer J1.22 (A3)
- net QR_5: now also J1.24 (A5); no longer J1.21 (A2)
- net QR_6: now also J1.25 (A6); no longer J1.20 (A1)
- net at J2.2, SW2.1 (A): now also C3.2
Other:
- note added: "Alimentacion +7,5v / Interruptor"
- note removed: "Alimentacion +7,5v"
- note removed: "Modulo QRE113"
- note removed: "Modulo Regulador 5v"
- note removed: "PINERAS -->"
- moved on the sheet: J2, P2, P3, P4, R1, R10, R11, R12, R2, R3, R4, R5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

Commit message: Agregue leds y actualice los pads del plaqueta mani
Parts:
- added LED1, LED2: LED, EESTN5:LED_1206, symbol EESTN5:LED
- added R13, R14: 330 ohm, symbol Device:R
Connections:
- net Earth: now also R13.1, R14.1
- net LED_2: now reaches J1.19 (A0)
- net LED_2: now also LED1.1 (A)
- net LED_1: now reaches J1.26 (A7)
- net LED_1: now also LED2.1 (A)
- new net: LED2.2 (K), R14.2
- new net: LED1.2 (K), R13.2
Other:
- note added: "S/Calibracion de Infrarrojo"
